File: smd-led-re450.kicad_pcb (KiCad board)
At the start: 2 copper layers, 23.4 x 20.3 mm, 14 parts, among them J1 Conn_01x08_Male, J2 Conn_01x04_Male

Commit message: Before resizing
Parts:
- moved R6 0.72 mm to (31.0, 35.6)
- moved R5 0.72 mm to (40.2, 37.1)
- turned DTop1 to 0 degrees
- turned R7 to 180 degrees
Connections:
- net +12V renamed /+
Routing:
- net /+: track 30.6 -> 47.5 mm, vias 2 -> 1
- net /Rli: track 0.00 -> 15.0 mm
- net /Wli: track 0.00 -> 13.7 mm
- net /S: track 0.00 -> 11.5 mm
- net /Rre: track 0.00 -> 7.92 mm
- net /Wt: track 0.00 -> 5.58 mm
- net Net-(DLinks1-Pad2): track 0.00 -> 5.51 mm
- net Net-(DSR1-Pad1): track 0.00 -> 3.18 mm
- net Net-(DSL1-Pad1): track 0.00 -> 2.69 mm
Other:
- board text added: "Re450 1.0"

Commit message: V1.1
Parts:
- J1: footprint Connector_PinHeader_1.27mm:PinHeader_1x08_P1.27mm_Vertical -> Connector_PinHeader_1.27mm:PinHeader_1x08_P1.27mm_Horizontal; moved to B.Cu
- J2: footprint Connector_PinHeader_1.27mm:PinHeader_1x04_P1.27mm_Vertical -> Connector_PinHeader_1.27mm:PinHeader_1x04_P1.27mm_Horizontal; moved to B.Cu
- R1: renamed from R5; value R -> 560; footprint Resistor_SMD:R_0603_1608Metric_Pad0.98x0.95mm_HandSolder -> Resistor_SMD:R_1206_3216Metric_Pad1.30x1.75mm_HandSolder
- R2: renamed from R6; value R -> 560; footprint Resistor_SMD:R_0603_1608Metric_Pad0.98x0.95mm_HandSolder -> Resistor_SMD:R_1206_3216Metric_Pad1.30x1.75mm_HandSolder
- R3: renamed from R1; value 800 -> 560; footprint Resistor_SMD:R_0603_1608Metric_Pad0.98x0.95mm_HandSolder -> Resistor_SMD:R_1206_3216Metric_Pad1.30x1.75mm_HandSolder
- R4: renamed from R2; value R -> 750; footprint Resistor_SMD:R_0603_1608Metric_Pad0.98x0.95mm_HandSolder -> Resistor_SMD:R_1206_3216Metric_Pad1.30x1.75mm_HandSolder
- R5: renamed from R7; value R -> 560; footprint Resistor_SMD:R_0603_1608Metric_Pad0.98x0.95mm_HandSolder -> Resistor_SMD:R_1206_3216Metric_Pad1.30x1.75mm_HandSolder
- R6: renamed from R3; value R -> 560; footprint Resistor_SMD:R_0603_1608Metric_Pad0.98x0.95mm_HandSolder -> Resistor_SMD:R_1206_3216Metric_Pad1.30x1.75mm_HandSolder
- R7: renamed from R4; value R -> 750; footprint Resistor_SMD:R_0603_1608Metric_Pad0.98x0.95mm_HandSolder -> Resistor_SMD:R_1206_3216Metric_Pad1.30x1.75mm_HandSolder
- moved J1 13.6 mm to (43.7, 37.6), turned to 90 degrees
- moved R4 12.8 mm to (39.6, 27.4)
- moved R6 12.7 mm to (30.5, 27.4), turned to 0 degrees
- moved R1 12.5 mm to (37.6, 24.9)
- moved R2 10.8 mm to (32.5, 24.9)
- moved R7 7.64 mm to (27.9, 30.0)
- moved R5 5.59 mm to (35.1, 30.0)
- moved R3 5.49 mm to (42.2, 30.0)
- moved J2 3.19 mm to (30.3, 37.6)
- turned DfL1 to -90 degrees
- turned DfR1 to -90 degrees
- turned HbL1 to -90 degrees
- turned HbR1 to -90 degrees
- renumbered DLinks1 to DfL1, DRechts1 to DfR1, DTop1 to DfT1, DSL1 to HbL1, DSR1 to HbR1
Connections:
- net /Wt renamed /FrT
- J1 pad 2: /Wre -> /FrL
- J1 pad 4: /Wli -> /FrR
- J1 pad 5: /S -> /BlL
- J1 pad 6: /Rli -> /BlR
- J1 pad 7: /Rre -> /HbL
- J1 pad 8: /+ -> /HbR
- J2 pad 1: /Wre -> /BlR
- J2 pad 2: /Wli -> /FrR
- J2 pad 3: /Rli -> /FrL
- R1 pad 2: /S -> /HbL
- R2 pad 2: /S -> /HbR
- R3 pad 2: /Wli -> /FrL
- R4 pad 2: /Rli -> /BlL
- R6 pad 2: /Wre -> /FrR
- R7 pad 2: /Rre -> /BlR
Routing:
- net /FrL: track 0.00 -> 23.7 mm
- net /FrR: track 0.00 -> 21.2 mm, vias 0 -> 1
- net /Wre: track 20.5 -> 0.00 mm
- net /BlR: track 0.00 -> 15.7 mm
- net /Rli: track 15.0 -> 0.00 mm
- net /Wli: track 13.7 -> 0.00 mm
- net /HbL: track 0.00 -> 13.2 mm
- net /HbR: track 0.00 -> 13.0 mm
- net /S: track 11.5 -> 0.00 mm
- net /BlL: track 0.00 -> 10.4 mm
- net /Rre: track 7.92 -> 0.00 mm
- net Net-(HbL1-Pad1): track 2.69 -> 10.1 mm
- net Net-(DfT1-Pad1): track 2.56 -> 9.25 mm
- net Net-(HbR1-Pad1): track 3.18 -> 9.76 mm
- net /FrT: track 5.58 -> 11.0 mm, vias 0 -> 1
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Other:
- outline, holes or cut-outs redrawn
- board text added: "Re450 1.1"
- board text removed: "Re450 1.0"
