File: smd-led-re450.kicad_sch (KiCad schematic)
At the start: 14 parts, among them J1 Conn_01x08_Male, J2 Conn_01x04_Male

Commit message: Before resizing
Connections:
- net +12V renamed +
Changed lines of the file:
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@@
   (junction (at 58.42 55.88) (diameter 0) (color 0 0 0 0)
   )
+  (junction (at 67.31 73.66) (diameter 0) (color 0 0 0 0)
+  )
+  (junction (at 144.78 55.88) (diameter 0) (color 0 0 0 0)
+  )
+  (junction (at 106.68 64.77) (diameter 0) (color 0 0 0 0)
+  )
+  (junction (at 68.58 91.44) (diameter 0) (color 0 0 0 0)
+  )
   (junction (at 67.31 64.77) (diameter 0) (color 0 0 0 0)
   )
-  (junction (at 77.47 64.77) (diameter 0) (color 0 0 0 0)
-  )
-  (junction (at 67.31 73.66) (diameter 0) (color 0 0 0 0)
-  )
-  (junction (at 144.78 55.88) (diameter 0) (color 0 0 0 0)
-  )
-  (junction (at 68.58 91.44) (diameter 0) (color 0 0 0 0)
-  )
-  (junction (at 106.68 64.77) (diameter 0) (color 0 0 0 0)
-  )
-  (wire (pts (xy 67.31 64.77) (xy 77.47 64.77))
-    (stroke (width 0) (type default) (color 0 0 0 0))
-  )
   (wire (pts (xy 113.03 82.55) (xy 121.92 82.55))
     (stroke (width 0) (type default) (color 0 0 0 0))
@@
     (stroke (width 0) (type default) (color 0 0 0 0))
   )
-  (wire (pts (xy 77.47 64.77) (xy 106.68 64.77))
-    (stroke (width 0) (type default) (color 0 0 0 0))
-  )
   (wire (pts (xy 106.68 50.8) (xy 106.68 64.77))
     (stroke (width 0) (type default) (color 0 0 0 0))
@@
   )
   (wire (pts (xy 67.31 73.66) (xy 74.93 73.66))
+    (stroke (width 0) (type default) (color 0 0 0 0))
+  )
+  (wire (pts (xy 67.31 64.77) (xy 106.68 64.77))
     (stroke (width 0) (type default) (color 0 0 0 0))
   )
@@
     (pin "1")
     (pin "2")
-  )
-  (symbol (lib_id "power:+12V") (at 77.47 64.77 0) (unit 1)
-    (in_bom yes) (on_board yes) (fields_autoplaced)
-    (property "Reference" "#PWR0101" (id 0) (at 77.47 68.58 0)
-      (effects (font (size 1.27 1.27)) hide)
-    )
-    (property "Value" "+12V" (id 1) (at 77.47 59.69 0))
-    (property "Footprint" "" (id 2) (at 77.47 64.77 0)
-      (effects (font (size 1.27 1.27)) hide)
-    )
-    (property "Datasheet" "" (id 3) (at 77.47 64.77 0)
-      (effects (font (size 1.27 1.27)) hide)
-    )
-    (pin "1")
   )
   (symbol (lib_id "Device:R") (at 77.47 55.88 90) (unit 1)
@@
   )
   (symbol_instances
-    (path "/8c858392-55bf-4c71-a37b-2dc92b7f753d"
-      (reference "#PWR0101") (unit 1) (value "+12V") (footprint "")
-    )
     (path "/35aa260c-35d5-4a9e-a5ce-23afedc1224d"
       (reference "DLinks1") (unit 1) (value "LED_Dual_AAKK_s") (footprint "LED_SMD:LED_0605_1613Metric")

Commit message: V1.1
Parts:
- J1: footprint Connector_PinHeader_1.27mm:PinHeader_1x08_P1.27mm_Vertical -> Connector_PinHeader_1.27mm:PinHeader_1x08_P1.27mm_Horizontal
- J2: footprint Connector_PinHeader_1.27mm:PinHeader_1x04_P1.27mm_Vertical -> Connector_PinHeader_1.27mm:PinHeader_1x04_P1.27mm_Horizontal
- R1: renamed from R5; value R -> 560; footprint Resistor_SMD:R_0603_1608Metric_Pad0.98x0.95mm_HandSolder -> Resistor_SMD:R_1206_3216Metric_Pad1.30x1.75mm_HandSolder
- R2: renamed from R6; value R -> 560; footprint Resistor_SMD:R_0603_1608Metric_Pad0.98x0.95mm_HandSolder -> Resistor_SMD:R_1206_3216Metric_Pad1.30x1.75mm_HandSolder
- R3: renamed from R1; value 800 -> 560; footprint Resistor_SMD:R_0603_1608Metric_Pad0.98x0.95mm_HandSolder -> Resistor_SMD:R_1206_3216Metric_Pad1.30x1.75mm_HandSolder
- R4: renamed from R2; value R -> 750; footprint Resistor_SMD:R_0603_1608Metric_Pad0.98x0.95mm_HandSolder -> Resistor_SMD:R_1206_3216Metric_Pad1.30x1.75mm_HandSolder
- R5: renamed from R7; value R -> 560; footprint Resistor_SMD:R_0603_1608Metric_Pad0.98x0.95mm_HandSolder -> Resistor_SMD:R_1206_3216Metric_Pad1.30x1.75mm_HandSolder
- R6: renamed from R3; value R -> 560; footprint Resistor_SMD:R_0603_1608Metric_Pad0.98x0.95mm_HandSolder -> Resistor_SMD:R_1206_3216Metric_Pad1.30x1.75mm_HandSolder
- R7: renamed from R4; value R -> 750; footprint Resistor_SMD:R_0603_1608Metric_Pad0.98x0.95mm_HandSolder -> Resistor_SMD:R_1206_3216Metric_Pad1.30x1.75mm_HandSolder
- renumbered DLinks1 to DfL1, DRechts1 to DfR1, DTop1 to DfT1, DSL1 to HbL1, DSR1 to HbR1
Connections:
- net +: no longer J1.8 (Pin_8)
- removed net Rli: J1.6 (Pin_6), J2.3 (Pin_3), R4.2
- net Rre renamed BlR
- net BlR: now also J1.6 (Pin_6), J2.1 (Pin_1); no longer J1.7 (Pin_7)
- removed net S: J1.5 (Pin_5), R1.2, R2.2
- net Wli renamed FrR
- net FrR: now also R6.2; no longer R3.2
- removed net Wre: J1.2 (Pin_2), J2.1 (Pin_1), R6.2
- net Wt renamed FrT
- new net BlL: J1.5 (Pin_5), R4.2
- new net FrL: J1.2 (Pin_2), J2.3 (Pin_3), R3.2
- new net HbL: J1.7 (Pin_7), R1.2
- new net HbR: J1.8 (Pin_8), R2.2
Other:
- note added: "Hb(R/L) = High Beam Left / Right FrR = Front Right FrT = Front Top FrL = Front Left BlR = Back Right BlL = Back Left"
- moved on the sheet: J2
